File: proto.kicad_pcb (KiCad board)
At the start: 2 copper layers, 329.4 x 130.6 mm, 146 parts, among them SW1 SW_Push, U1 ATmega32U4-AU, Y1 16MHz

Commit message: rotary
Parts:
- removed D62: S0D-123, Diode_SMD:D_SOD-123
- removed MX62: MX-NoLED, MX_Alps_Hybrid:MX-1U
- added C8: 100nF, Capacitor_SMD:C_0805_2012Metric, B.Cu at (180.8, 114.8)
- added C9: 100nF, Capacitor_SMD:C_0805_2012Metric, B.Cu at (175.8, 114.8)
- added SW2: Rotary_Encoder_Switch, Rotary_Encoder:RotaryEncoder_Alps_EC11E-Switch_Vertical_H20mm, F.Cu at (180.8, 120.4)
- moved R3 190.9 mm to (53.3, 156.2)
- moved Y1 190.9 mm to (53.3, 142.2)
- moved C1 190.9 mm to (53.3, 137.2)
- moved C2 190.9 mm to (53.3, 147.3)
- moved C3 190.9 mm to (63.5, 151.1)
- moved C4 190.9 mm to (58.4, 151.1)
- moved C5 190.9 mm to (59.7, 133.3)
- moved D1 190.9 mm to (21.2, 53.4)
- moved D10 190.9 mm to (214.9, 63.1)
- moved D11 190.9 mm to (233.8, 60.7)
- moved D12 190.9 mm to (252.7, 58.4)
- moved D13 190.9 mm to (271.6, 56.1)
- moved D14 190.9 mm to (290.5, 53.8)
- moved D15 190.9 mm to (309.4, 51.5)
- moved D16 190.9 mm to (18.8, 72.3)
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Connections:
- U1 pad 11: Net-(U1-Pad11) -> ROT1
- U1 pad 12: Net-(U1-Pad12) -> ROT0
Routing:
- net ROT0: track 0.00 -> 202.7 mm, vias 0 -> 2
- net ROT1: track 0.00 -> 202.7 mm, vias 0 -> 2
- net COL7: track 196.3 -> 211.2 mm
- net GND: track 243.7 -> 254.8 mm
- net ROW4: track 137.1 -> 146.6 mm
- net Net-(D62-Pad2): track 6.30 -> 0.00 mm
- net COL10: track 241.7 -> 243.2 mm
- added copper zone on B.Cu, net GND
Other:
- board size 329.4 x 130.6 mm -> 329.3 x 130.6 mm
- board text added: "wings"

Commit message: edits
Parts:
- moved C5 0.63 mm to (59.1, 133.3), turned to 270 degrees
Routing:
- net COL11: track 202.1 -> 263.8 mm
- net +5V: track 81.0 -> 98.0 mm, vias 4 -> 8
- net COL7: track 211.2 -> 222.1 mm
- net COL6: track 179.2 -> 189.8 mm
- net COL1: track 119.1 -> 128.6 mm
- net COL2: track 101.1 -> 109.7 mm
- net COL4: track 88.6 -> 96.4 mm
- net COL0: track 141.3 -> 148.8 mm
- net COL3: track 85.4 -> 92.5 mm
- net COL5: track 106.5 -> 113.3 mm
- net COL14: track 322.5 -> 329.0 mm
- net GND: track 254.8 -> 260.5 mm
- net COL10: track 243.2 -> 248.1 mm
- net ROW2: track 377.2 -> 372.9 mm
- net COL13: track 302.2 -> 306.2 mm
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