File: proto.kicad_pcb (KiCad board)
At the start: 2 copper layers, 329.3 x 130.6 mm, 147 parts, among them SW1 SW_Push, SW2 Rotary_Encoder_Switch, U1 ATmega32U4-AU, Y1 16MHz

Commit message: plate stl, updated pcb
Parts:
- moved C9 2.15 mm to (174.0, 115.9)
- moved C8 2.09 mm to (179.1, 115.9)
- moved SW2 1.89 mm to (179.0, 120.9)
Routing:
- net GND: track 260.5 -> 256.4 mm
- net ROT1: track 202.7 -> 204.5 mm
- net ROW4: track 146.6 -> 144.8 mm
- net COL7: track 222.1 -> 220.8 mm
- net ROT0: track 202.7 -> 203.7 mm
